Commit message: Release Robotrola Core as complete open research humanoid platform
Ship 42-DOF description, pure-Python safety path, MCU and motor-bridge
firmware sources, BOM stage cost model, protocol sim, diligence demo,
claims matrix, and Apache/CERN-OHL licenses. Public-ready README and CI
gates for technical due diligence without hardware.

File: cad/urdf/robotrola_r01_reference.urdf.xacro (robot description, xacro)
@@ -2,14 +2,436 @@
 <robot name="robotrola_r01" xmlns:xacro="http://www.ros.org/wiki/xacro">
   <xacro:property name="mesh_prefix" value="package://robotrola_description/meshes" />
+  <!-- Robotrola R-01 full-body research description: 42 revolute DOF -->
   <link name="base_link"/>
-  <link name="pelvis_link"><visual><geometry><mesh filename="${mesh_prefix}/pelvis_frame.stl" scale="0.001 0.001 0.001"/></geometry></visual></link>
-  <joint name="base_to_pelvis" type="fixed"><parent link="base_link"/><child link="pelvis_link"/><origin xyz="0 0 0.9" rpy="0 0 0"/></joint>
-  <link name="torso_link"><visual><geometry><mesh filename="${mesh_prefix}/torso_front_shell.stl" scale="0.001 0.001 0.001"/></geometry></visual></link>
-  <joint name="pelvis_to_torso" type="fixed"><parent link="pelvis_link"/><child link="torso_link"/><origin xyz="0 0 0.25" rpy="0 0 0"/></joint>
-  <link name="head_link"><visual><geometry><mesh filename="${mesh_prefix}/head_shell_front.stl" scale="0.001 0.001 0.001"/></geometry></visual></link>
-  <joint name="neck_yaw" type="revolute"><parent link="torso_link"/><child link="head_link"/><origin xyz="0 0 0.34" rpy="0 0 0"/><axis xyz="0 0 1"/><limit lower="-0.9" upper="0.9" effort="0.5" velocity="0.25"/></joint>
-  <link name="left_upper_arm_link"><visual><geometry><mesh filename="${mesh_prefix}/upper_arm_shell.stl" scale="0.001 0.001 0.001"/></geometry></visual></link>
-  <joint name="left_shoulder_pitch" type="revolute"><parent link="torso_link"/><child link="left_upper_arm_link"/><origin xyz="0.16 0 0.21" rpy="0 0 0"/><axis xyz="1 0 0"/><limit lower="-1.2" upper="1.2" effort="1.2" velocity="0.2"/></joint>
-  <link name="left_forearm_link"><visual><geometry><mesh filename="${mesh_prefix}/forearm_shell.stl" scale="0.001 0.001 0.001"/></geometry></visual></link>
-  <joint name="left_elbow" type="revolute"><parent link="left_upper_arm_link"/><child link="left_forearm_link"/><origin xyz="0 0 -0.18" rpy="0 0 0"/><axis xyz="1 0 0"/><limit lower="0" upper="2.1" effort="0.8" velocity="0.25"/></joint>
+  <link name="pelvis_link">
+    <visual><geometry><mesh filename="${mesh_prefix}/pelvis_frame.stl" scale="0.001 0.001 0.001"/></geometry></visual>
+    <collision><geometry><box size="0.25 0.2 0.12"/></geometry></collision>
+  </link>
+  <joint name="base_to_pelvis" type="fixed">
+    <parent link="base_link"/><child link="pelvis_link"/>
+    <origin xyz="0 0 0.95" rpy="0 0 0"/>
+  </joint>
+  <link name="waist_link">
+    <visual><geometry><mesh filename="${mesh_prefix}/pelvis_frame.stl" scale="0.001 0.001 0.001"/></geometry></visual>
+    <collision><geometry><cylinder radius="0.04" length="0.08"/></geometry></collision>
+  </link>
+  <joint name="waist_yaw" type="revolute">
+    <parent link="pelvis_link"/><child link="waist_link"/>
+    <origin xyz="0 0 0.08" rpy="0 0 0"/>
+    <axis xyz="0 0 1"/>
+    <limit lower="-0.6" upper="0.6" effort="2.0" velocity="0.2"/>
+  </joint>
+  <link name="torso_link">
+    <visual><geometry><mesh filename="${mesh_prefix}/torso_front_shell.stl" scale="0.001 0.001 0.001"/></geometry></visual>
+    <collision><geometry><cylinder radius="0.04" length="0.08"/></geometry></collision>
+  </link>
+  <joint name="waist_pitch" type="revolute">
+    <parent link="waist_link"/><child link="torso_link"/>
+    <origin xyz="0 0 0.12" rpy="0 0 0"/>
+    <axis xyz="0 1 0"/>
+    <limit lower="-0.35" upper="0.45" effort="2.5" velocity="0.2"/>
+  </joint>
+  <link name="torso_roll_link">
+    <visual><geometry><mesh filename="${mesh_prefix}/torso_back_shell.stl" scale="0.001 0.001 0.001"/></geometry></visual>
+    <collision><geometry><cylinder radius="0.04" length="0.08"/></geometry></collision>
+  </link>
+  <joint name="waist_roll" type="revolute">
+    <parent link="torso_link"/><child link="torso_roll_link"/>
+    <origin xyz="0 0 0.05" rpy="0 0 0"/>
+    <axis xyz="1 0 0"/>
+    <limit lower="-0.3" upper="0.3" effort="1.5" velocity="0.2"/>
+  </joint>
+  <link name="neck_yaw_link">
+    <visual><geometry><mesh filename="${mesh_prefix}/neck_gimbal_mount.stl" scale="0.001 0.001 0.001"/></geometry></visual>
+    <collision><geometry><cylinder radius="0.04" length="0.08"/></geometry></collision>
+  </link>
+  <joint name="neck_yaw" type="revolute">
+    <parent link="torso_roll_link"/><child link="neck_yaw_link"/>
+    <origin xyz="0 0 0.28" rpy="0 0 0"/>
+    <axis xyz="0 0 1"/>
+    <limit lower="-0.9" upper="0.9" effort="0.5" velocity="0.25"/>
+  </joint>
+  <link name="neck_pitch_link"/>
+  <joint name="neck_pitch" type="revolute">
+    <parent link="neck_yaw_link"/><child link="neck_pitch_link"/>
+    <origin xyz="0 0 0.04" rpy="0 0 0"/>
+    <axis xyz="0 1 0"/>
+    <limit lower="-0.5" upper="0.6" effort="0.5" velocity="0.25"/>
+  </joint>
+  <link name="head_link">
+    <visual><geometry><mesh filename="${mesh_prefix}/head_shell_front.stl" scale="0.001 0.001 0.001"/></geometry></visual>
+    <collision><geometry><cylinder radius="0.04" length="0.08"/></geometry></collision>
+  </link>
+  <joint name="neck_roll" type="revolute">
+    <parent link="neck_pitch_link"/><child link="head_link"/>
+    <origin xyz="0 0 0.06" rpy="0 0 0"/>
+    <axis xyz="1 0 0"/>
+    <limit lower="-0.35" upper="0.35" effort="0.4" velocity="0.2"/>
+  </joint>
+  <link name="left_shoulder_pitch_link">
+    <visual><geometry><mesh filename="${mesh_prefix}/upper_arm_shell.stl" scale="0.001 0.001 0.001"/></geometry></visual>
+    <collision><geometry><cylinder radius="0.04" length="0.08"/></geometry></collision>
+  </link>
+  <joint name="left_shoulder_pitch" type="revolute">
+    <parent link="torso_roll_link"/><child link="left_shoulder_pitch_link"/>
+    <origin xyz="0.18 0 0.22" rpy="0 0 0"/>
+    <axis xyz="0 1 0"/>
+    <limit lower="-1.4" upper="1.4" effort="1.5" velocity="0.25"/>
+  </joint>
+  <link name="left_shoulder_roll_link"/>
+  <joint name="left_shoulder_roll" type="revolute">
+    <parent link="left_shoulder_pitch_link"/><child link="left_shoulder_roll_link"/>
+    <origin xyz="0 0 0" rpy="0 0 0"/>
+    <axis xyz="1 0 0"/>
+    <limit lower="-0.3" upper="1.5" effort="1.2" velocity="0.25"/>
+  </joint>
+  <link name="left_upper_arm_link"/>
+  <joint name="left_shoulder_yaw" type="revolute">
+    <parent link="left_shoulder_roll_link"/><child link="left_upper_arm_link"/>
+    <origin xyz="0 0 -0.05" rpy="0 0 0"/>
+    <axis xyz="0 0 1"/>
+    <limit lower="-1.2" upper="1.2" effort="1.0" velocity="0.3"/>
+  </joint>
+  <link name="left_forearm_link">
+    <visual><geometry><mesh filename="${mesh_prefix}/forearm_shell.stl" scale="0.001 0.001 0.001"/></geometry></visual>
+    <collision><geometry><cylinder radius="0.04" length="0.08"/></geometry></collision>
+  </link>
+  <joint name="left_elbow" type="revolute">
+    <parent link="left_upper_arm_link"/><child link="left_forearm_link"/>
+    <origin xyz="0 0 -0.22" rpy="0 0 0"/>
+    <axis xyz="0 1 0"/>
+    <limit lower="0.0" upper="2.2" effort="1.0" velocity="0.3"/>
+  </joint>
+  <link name="left_wrist_yaw_link"/>
+  <joint name="left_wrist_yaw" type="revolute">
+    <parent link="left_forearm_link"/><child link="left_wrist_yaw_link"/>
+    <origin xyz="0 0 -0.2" rpy="0 0 0"/>
+    <axis xyz="0 0 1"/>
+    <limit lower="-1.4" upper="1.4" effort="0.4" velocity="0.4"/>
+  </joint>
+  <link name="left_wrist_pitch_link"/>
+  <joint name="left_wrist_pitch" type="revolute">
+    <parent link="left_wrist_yaw_link"/><child link="left_wrist_pitch_link"/>
+    <origin xyz="0 0 0" rpy="0 0 0"/>
+    <axis xyz="0 1 0"/>
+    <limit lower="-0.9" upper="0.9" effort="0.4" velocity="0.4"/>
+  </joint>
+  <link name="left_hand_link">
+    <visual><geometry><mesh filename="${mesh_prefix}/hand_palm.stl" scale="0.001 0.001 0.001"/></geometry></visual>
+    <collision><geometry><cylinder radius="0.04" length="0.08"/></geometry></collision>
+  </link>
+  <joint name="left_wrist_roll" type="revolute">
+    <parent link="left_wrist_pitch_link"/><child link="left_hand_link"/>
+    <origin xyz="0 0 0" rpy="0 0 0"/>
+    <axis xyz="1 0 0"/>
+    <limit lower="-0.9" upper="0.9" effort="0.3" velocity="0.4"/>
+  </joint>
+  <link name="left_thumb_link">
+    <visual><geometry><mesh filename="${mesh_prefix}/finger_phalanx_proximal.stl" scale="0.001 0.001 0.001"/></geometry></visual>
+    <collision><geometry><cylinder radius="0.04" length="0.08"/></geometry></collision>
+  </link>
+  <joint name="left_thumb_curl" type="revolute">
+    <parent link="left_hand_link"/><child link="left_thumb_link"/>
+    <origin xyz="-0.04 0.03 0.02" rpy="0 0 0"/>
+    <axis xyz="0 1 0"/>
+    <limit lower="0.0" upper="1.4" effort="0.15" velocity="0.5"/>
+  </joint>
+  <link name="left_index_link">
+    <visual><geometry><mesh filename="${mesh_prefix}/finger_phalanx_proximal.stl" scale="0.001 0.001 0.001"/></geometry></visual>
+    <collision><geometry><cylinder radius="0.04" length="0.08"/></geometry></collision>
+  </link>
+  <joint name="left_index_curl" type="revolute">
+    <parent link="left_hand_link"/><child link="left_index_link"/>
+    <origin xyz="-0.02 0.03 0.02" rpy="0 0 0"/>
+    <axis xyz="0 1 0"/>
+    <limit lower="0.0" upper="1.4" effort="0.15" velocity="0.5"/>
+  </joint>
+  <link name="left_middle_link">
+    <visual><geometry><mesh filename="${mesh_prefix}/finger_phalanx_distal.stl" scale="0.001 0.001 0.001"/></geometry></visual>
+    <collision><geometry><cylinder radius="0.04" length="0.08"/></geometry></collision>
+  </link>
+  <joint name="left_middle_curl" type="revolute">
+    <parent link="left_hand_link"/><child link="left_middle_link"/>
+    <origin xyz="0.0 0.03 0.02" rpy="0 0 0"/>
+    <axis xyz="0 1 0"/>
+    <limit lower="0.0" upper="1.4" effort="0.15" velocity="0.5"/>
+  </joint>
+  <link name="left_ring_link">
+    <visual><geometry><mesh filename="${mesh_prefix}/finger_phalanx_distal.stl" scale="0.001 0.001 0.001"/></geometry></visual>
+    <collision><geometry><cylinder radius="0.04" length="0.08"/></geometry></collision>
+  </link>
+  <joint name="left_ring_curl" type="revolute">
+    <parent link="left_hand_link"/><child link="left_ring_link"/>
+    <origin xyz="0.02 0.03 0.02" rpy="0 0 0"/>
+    <axis xyz="0 1 0"/>
+    <limit lower="0.0" upper="1.4" effort="0.15" velocity="0.5"/>
+  </joint>
+  <link name="left_pinky_link">
+    <visual><geometry><mesh filename="${mesh_prefix}/finger_phalanx_distal.stl" scale="0.001 0.001 0.001"/></geometry></visual>
+    <collision><geometry><cylinder radius="0.04" length="0.08"/></geometry></collision>
+  </link>
+  <joint name="left_pinky_curl" type="revolute">
+    <parent link="left_hand_link"/><child link="left_pinky_link"/>
+    <origin xyz="0.04 0.03 0.02" rpy="0 0 0"/>
+    <axis xyz="0 1 0"/>
+    <limit lower="0.0" upper="1.4" effort="0.15" velocity="0.5"/>
+  </joint>
+  <link name="right_shoulder_pitch_link">
+    <visual><geometry><mesh filename="${mesh_prefix}/upper_arm_shell.stl" scale="0.001 0.001 0.001"/></geometry></visual>
+    <collision><geometry><cylinder radius="0.04" length="0.08"/></geometry></collision>
+  </link>
+  <joint name="right_shoulder_pitch" type="revolute">
+    <parent link="torso_roll_link"/><child link="right_shoulder_pitch_link"/>
+    <origin xyz="-0.18 0 0.22" rpy="0 0 0"/>
+    <axis xyz="0 1 0"/>
+    <limit lower="-1.4" upper="1.4" effort="1.5" velocity="0.25"/>
+  </joint>
+  <link name="right_shoulder_roll_link"/>
+  <joint name="right_shoulder_roll" type="revolute">
+    <parent link="right_shoulder_pitch_link"/><child link="right_shoulder_roll_link"/>
+    <origin xyz="0 0 0" rpy="0 0 0"/>
+    <axis xyz="1 0 0"/>
+    <limit lower="-1.5" upper="0.3" effort="1.2" velocity="0.25"/>
+  </joint>
+  <link name="right_upper_arm_link"/>
+  <joint name="right_shoulder_yaw" type="revolute">
+    <parent link="right_shoulder_roll_link"/><child link="right_upper_arm_link"/>
+    <origin xyz="0 0 -0.05" rpy="0 0 0"/>
+    <axis xyz="0 0 1"/>
+    <limit lower="-1.2" upper="1.2" effort="1.0" velocity="0.3"/>
+  </joint>
+  <link name="right_forearm_link">
+    <visual><geometry><mesh filename="${mesh_prefix}/forearm_shell.stl" scale="0.001 0.001 0.001"/></geometry></visual>
+    <collision><geometry><cylinder radius="0.04" length="0.08"/></geometry></collision>
+  </link>
+  <joint name="right_elbow" type="revolute">
+    <parent link="right_upper_arm_link"/><child link="right_forearm_link"/>
+    <origin xyz="0 0 -0.22" rpy="0 0 0"/>
+    <axis xyz="0 1 0"/>
+    <limit lower="0.0" upper="2.2" effort="1.0" velocity="0.3"/>
+  </joint>
+  <link name="right_wrist_yaw_link"/>
+  <joint name="right_wrist_yaw" type="revolute">
+    <parent link="right_forearm_link"/><child link="right_wrist_yaw_link"/>
+    <origin xyz="0 0 -0.2" rpy="0 0 0"/>
+    <axis xyz="0 0 1"/>
+    <limit lower="-1.4" upper="1.4" effort="0.4" velocity="0.4"/>
+  </joint>
+  <link name="right_wrist_pitch_link"/>
+  <joint name="right_wrist_pitch" type="revolute">
+    <parent link="right_wrist_yaw_link"/><child link="right_wrist_pitch_link"/>
+    <origin xyz="0 0 0" rpy="0 0 0"/>
+    <axis xyz="0 1 0"/>
+    <limit lower="-0.9" upper="0.9" effort="0.4" velocity="0.4"/>
+  </joint>
+  <link name="right_hand_link">
+    <visual><geometry><mesh filename="${mesh_prefix}/hand_palm.stl" scale="0.001 0.001 0.001"/></geometry></visual>
+    <collision><geometry><cylinder radius="0.04" length="0.08"/></geometry></collision>
+  </link>
+  <joint name="right_wrist_roll" type="revolute">
+    <parent link="right_wrist_pitch_link"/><child link="right_hand_link"/>
+    <origin xyz="0 0 0" rpy="0 0 0"/>
+    <axis xyz="1 0 0"/>
+    <limit lower="-0.9" upper="0.9" effort="0.3" velocity="0.4"/>
+  </joint>
+  <link name="right_thumb_link">
+    <visual><geometry><mesh filename="${mesh_prefix}/finger_phalanx_proximal.stl" scale="0.001 0.001 0.001"/></geometry></visual>
+    <collision><geometry><cylinder radius="0.04" length="0.08"/></geometry></collision>
+  </link>
+  <joint name="right_thumb_curl" type="revolute">
+    <parent link="right_hand_link"/><child link="right_thumb_link"/>
+    <origin xyz="-0.04 0.03 0.02" rpy="0 0 0"/>
+    <axis xyz="0 1 0"/>
+    <limit lower="0.0" upper="1.4" effort="0.15" velocity="0.5"/>
+  </joint>
+  <link name="right_index_link">
+    <visual><geometry><mesh filename="${mesh_prefix}/finger_phalanx_proximal.stl" scale="0.001 0.001 0.001"/></geometry></visual>
+    <collision><geometry><cylinder radius="0.04" length="0.08"/></geometry></collision>
+  </link>
+  <joint name="right_index_curl" type="revolute">
+    <parent link="right_hand_link"/><child link="right_index_link"/>
+    <origin xyz="-0.02 0.03 0.02" rpy="0 0 0"/>
+    <axis xyz="0 1 0"/>
+    <limit lower="0.0" upper="1.4" effort="0.15" velocity="0.5"/>
+  </joint>
+  <link name="right_middle_link">
+    <visual><geometry><mesh filename="${mesh_prefix}/finger_phalanx_distal.stl" scale="0.001 0.001 0.001"/></geometry></visual>
+    <collision><geometry><cylinder radius="0.04" length="0.08"/></geometry></collision>
+  </link>
+  <joint name="right_middle_curl" type="revolute">
+    <parent link="right_hand_link"/><child link="right_middle_link"/>
+    <origin xyz="0.0 0.03 0.02" rpy="0 0 0"/>
+    <axis xyz="0 1 0"/>
+    <limit lower="0.0" upper="1.4" effort="0.15" velocity="0.5"/>
+  </joint>
+  <link name="right_ring_link">
+    <visual><geometry><mesh filename="${mesh_prefix}/finger_phalanx_distal.stl" scale="0.001 0.001 0.001"/></geometry></visual>
+    <collision><geometry><cylinder radius="0.04" length="0.08"/></geometry></collision>
+  </link>
+  <joint name="right_ring_curl" type="revolute">
+    <parent link="right_hand_link"/><child link="right_ring_link"/>
+    <origin xyz="0.02 0.03 0.02" rpy="0 0 0"/>
+    <axis xyz="0 1 0"/>
+    <limit lower="0.0" upper="1.4" effort="0.15" velocity="0.5"/>
+  </joint>
+  <link name="right_pinky_link">
+    <visual><geometry><mesh filename="${mesh_prefix}/finger_phalanx_distal.stl" scale="0.001 0.001 0.001"/></geometry></visual>
+    <collision><geometry><cylinder radius="0.04" length="0.08"/></geometry></collision>
+  </link>
+  <joint name="right_pinky_curl" type="revolute">
+    <parent link="right_hand_link"/><child link="right_pinky_link"/>
+    <origin xyz="0.04 0.03 0.02" rpy="0 0 0"/>
+    <axis xyz="0 1 0"/>
+    <limit lower="0.0" upper="1.4" effort="0.15" velocity="0.5"/>
+  </joint>
+  <link name="left_hip_yaw_link"/>
+  <joint name="left_hip_yaw" type="revolute">
+    <parent link="pelvis_link"/><child link="left_hip_yaw_link"/>
+    <origin xyz="0 0.1 -0.05" rpy="0 0 0"/>
+    <axis xyz="0 0 1"/>
+    <limit lower="-0.6" upper="0.6" effort="2.0" velocity="0.25"/>
+  </joint>
+  <link name="left_hip_roll_link"/>
+  <joint name="left_hip_roll" type="revolute">
+    <parent link="left_hip_yaw_link"/><child link="left_hip_roll_link"/>
+    <origin xyz="0 0 0" rpy="0 0 0"/>
+    <axis xyz="1 0 0"/>
+    <limit lower="-0.4" upper="0.4" effort="2.0" velocity="0.25"/>
+  </joint>
+  <link name="left_thigh_link">
+    <visual><geometry><mesh filename="${mesh_prefix}/thigh_shell.stl" scale="0.001 0.001 0.001"/></geometry></visual>
+    <collision><geometry><cylinder radius="0.04" length="0.08"/></geometry></collision>
+  </link>
+  <joint name="left_hip_pitch" type="revolute">
+    <parent link="left_hip_roll_link"/><child link="left_thigh_link"/>
+    <origin xyz="0 0 0" rpy="0 0 0"/>
+    <axis xyz="0 1 0"/>
+    <limit lower="-1.4" upper="0.8" effort="3.0" velocity="0.25"/>
+  </joint>
+  <link name="left_shin_link">
+    <visual><geometry><mesh filename="${mesh_prefix}/shin_shell.stl" scale="0.001 0.001 0.001"/></geometry></visual>
+    <collision><geometry><cylinder radius="0.04" length="0.08"/></geometry></collision>
+  </link>
+  <joint name="left_knee" type="revolute">
+    <parent link="left_thigh_link"/><child link="left_shin_link"/>
+    <origin xyz="0 0 -0.35" rpy="0 0 0"/>
+    <axis xyz="0 1 0"/>
+    <limit lower="0.0" upper="2.2" effort="3.0" velocity="0.3"/>
+  </joint>
+  <link name="left_ankle_pitch_link"/>
+  <joint name="left_ankle_pitch" type="revolute">
+    <parent link="left_shin_link"/><child link="left_ankle_pitch_link"/>
+    <origin xyz="0 0 -0.35" rpy="0 0 0"/>
+    <axis xyz="0 1 0"/>
+    <limit lower="-0.7" upper="0.7" effort="1.5" velocity="0.3"/>
+  </joint>
+  <link name="left_foot_link">
+    <visual><geometry><mesh filename="${mesh_prefix}/foot_sole_force_sensor_mount.stl" scale="0.001 0.001 0.001"/></geometry></visual>
+    <collision><geometry><cylinder radius="0.04" length="0.08"/></geometry></collision>
+  </link>
+  <joint name="left_ankle_roll" type="revolute">
+    <parent link="left_ankle_pitch_link"/><child link="left_foot_link"/>
+    <origin xyz="0 0 0" rpy="0 0 0"/>
+    <axis xyz="1 0 0"/>
+    <limit lower="-0.4" upper="0.4" effort="1.0" velocity="0.3"/>
+  </joint>
+  <link name="right_hip_yaw_link"/>
+  <joint name="right_hip_yaw" type="revolute">
+    <parent link="pelvis_link"/><child link="right_hip_yaw_link"/>
+    <origin xyz="0 -0.1 -0.05" rpy="0 0 0"/>
+    <axis xyz="0 0 1"/>
+    <limit lower="-0.6" upper="0.6" effort="2.0" velocity="0.25"/>
+  </joint>
+  <link name="right_hip_roll_link"/>
+  <joint name="right_hip_roll" type="revolute">
+    <parent link="right_hip_yaw_link"/><child link="right_hip_roll_link"/>
+    <origin xyz="0 0 0" rpy="0 0 0"/>
+    <axis xyz="1 0 0"/>
+    <limit lower="-0.4" upper="0.4" effort="2.0" velocity="0.25"/>
+  </joint>
+  <link name="right_thigh_link">
+    <visual><geometry><mesh filename="${mesh_prefix}/thigh_shell.stl" scale="0.001 0.001 0.001"/></geometry></visual>
+    <collision><geometry><cylinder radius="0.04" length="0.08"/></geometry></collision>
+  </link>
+  <joint name="right_hip_pitch" type="revolute">
+    <parent link="right_hip_roll_link"/><child link="right_thigh_link"/>
+    <origin xyz="0 0 0" rpy="0 0 0"/>
+    <axis xyz="0 1 0"/>
+    <limit lower="-1.4" upper="0.8" effort="3.0" velocity="0.25"/>
+  </joint>
+  <link name="right_shin_link">
+    <visual><geometry><mesh filename="${mesh_prefix}/shin_shell.stl" scale="0.001 0.001 0.001"/></geometry></visual>
+    <collision><geometry><cylinder radius="0.04" length="0.08"/></geometry></collision>
+  </link>
+  <joint name="right_knee" type="revolute">
+    <parent link="right_thigh_link"/><child link="right_shin_link"/>
+    <origin xyz="0 0 -0.35" rpy="0 0 0"/>
+    <axis xyz="0 1 0"/>
+    <limit lower="0.0" upper="2.2" effort="3.0" velocity="0.3"/>
+  </joint>
+  <link name="right_ankle_pitch_link"/>
+  <joint name="right_ankle_pitch" type="revolute">
+    <parent link="right_shin_link"/><child link="right_ankle_pitch_link"/>
+    <origin xyz="0 0 -0.35" rpy="0 0 0"/>
+    <axis xyz="0 1 0"/>
+    <limit lower="-0.7" upper="0.7" effort="1.5" velocity="0.3"/>
+  </joint>
+  <link name="right_foot_link">
+    <visual><geometry><mesh filename="${mesh_prefix}/foot_sole_force_sensor_mount.stl" scale="0.001 0.001 0.001"/></geometry></visual>
+    <collision><geometry><cylinder radius="0.04" length="0.08"/></geometry></collision>
+  </link>
+  <joint name="right_ankle_roll" type="revolute">
+    <parent link="right_ankle_pitch_link"/><child link="right_foot_link"/>
+    <origin xyz="0 0 0" rpy="0 0 0"/>
+    <axis xyz="1 0 0"/>
+    <limit lower="-0.4" upper="0.4" effort="1.0" velocity="0.3"/>
+  </joint>
+  <link name="camera_bar_link">
+    <visual><geometry><mesh filename="${mesh_prefix}/camera_bar_mount.stl" scale="0.001 0.001 0.001"/></geometry></visual>
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