Commit message: Ship Phase-0+ open research core: honesty, joint filter, ROS nodes, sim smoke.
Rename safety MCU package to esp32_safety_mcu (serial, not micro-ROS), add estimated URDF inertias, dual-license pointer, and LeRobot v3-layout export. Replace empty ROS shells with filter/teleop/perception nodes, shared joint_filter, sim_smoke and firmware gates, and extend CI/SPEC/CLAIMS for the new diligence bar.

File: cad/urdf/robotrola_r01_reference.urdf.xacro (robot description, xacro)
@@ -3,6 +3,20 @@
   <xacro:property name="mesh_prefix" value="package://robotrola_description/meshes" />
   <!-- Robotrola R-01 full-body research description: 42 revolute DOF -->
-  <link name="base_link"/>
+  <!-- Inertial blocks are ESTIMATED (engineering placeholders), not measured hardware. -->
+  <link name="base_link">
+    <!-- ESTIMATED inertia (not measured hardware) -->
+    <inertial>
+      <origin xyz="0 0 0" rpy="0 0 0"/>
+      <mass value="0.01"/>
+      <inertia ixx="1e-05" ixy="0" ixz="0" iyy="1e-05" iyz="0" izz="1e-05"/>
+    </inertial>
+  </link>
   <link name="pelvis_link">
+    <!-- ESTIMATED inertia (not measured hardware) -->
+    <inertial>
+      <origin xyz="0 0 0" rpy="0 0 0"/>
+      <mass value="8.0"/>
+      <inertia ixx="0.08" ixy="0" ixz="0" iyy="0.06" iyz="0" izz="0.05"/>
+    </inertial>
     <visual><geometry><mesh filename="${mesh_prefix}/pelvis_frame.stl" scale="0.001 0.001 0.001"/></geometry></visual>
     <collision><geometry><box size="0.25 0.2 0.12"/></geometry></collision>
@@ -13,4 +27,10 @@
   </joint>
   <link name="waist_link">
+    <!-- ESTIMATED inertia (not measured hardware) -->
+    <inertial>
+      <origin xyz="0 0 0" rpy="0 0 0"/>
+      <mass value="2.5"/>
+      <inertia ixx="0.02" ixy="0" ixz="0" iyy="0.015" iyz="0" izz="0.012"/>
+    </inertial>
     <visual><geometry><mesh filename="${mesh_prefix}/pelvis_frame.stl" scale="0.001 0.001 0.001"/></geometry></visual>
     <collision><geometry><cylinder radius="0.04" length="0.08"/></geometry></collision>
@@ -23,4 +43,10 @@
   </joint>
   <link name="torso_link">
+    <!-- ESTIMATED inertia (not measured hardware) -->
+    <inertial>
+      <origin xyz="0 0 0" rpy="0 0 0"/>
+      <mass value="6.0"/>
+      <inertia ixx="0.1" ixy="0" ixz="0" iyy="0.08" iyz="0" izz="0.05"/>
+    </inertial>
     <visual><geometry><mesh filename="${mesh_prefix}/torso_front_shell.stl" scale="0.001 0.001 0.001"/></geometry></visual>
     <collision><geometry><cylinder radius="0.04" length="0.08"/></geometry></collision>
@@ -33,4 +59,10 @@
   </joint>
   <link name="torso_roll_link">
+    <!-- ESTIMATED inertia (not measured hardware) -->
+    <inertial>
+      <origin xyz="0 0 0" rpy="0 0 0"/>
+      <mass value="6.0"/>
+      <inertia ixx="0.1" ixy="0" ixz="0" iyy="0.08" iyz="0" izz="0.05"/>
+    </inertial>
     <visual><geometry><mesh filename="${mesh_prefix}/torso_back_shell.stl" scale="0.001 0.001 0.001"/></geometry></visual>
     <collision><geometry><cylinder radius="0.04" length="0.08"/></geometry></collision>
@@ -43,4 +75,10 @@
   </joint>
   <link name="neck_yaw_link">
+    <!-- ESTIMATED inertia (not measured hardware) -->
+    <inertial>
+      <origin xyz="0 0 0" rpy="0 0 0"/>
+      <mass value="0.4"/>
+      <inertia ixx="0.001" ixy="0" ixz="0" iyy="0.001" iyz="0" izz="0.0008"/>
+    </inertial>
     <visual><geometry><mesh filename="${mesh_prefix}/neck_gimbal_mount.stl" scale="0.001 0.001 0.001"/></geometry></visual>
     <collision><geometry><cylinder radius="0.04" length="0.08"/></geometry></collision>
@@ -52,5 +90,12 @@
     <limit lower="-0.9" upper="0.9" effort="0.5" velocity="0.25"/>
   </joint>
-  <link name="neck_pitch_link"/>
+  <link name="neck_pitch_link">
+    <!-- ESTIMATED inertia (not measured hardware) -->
+    <inertial>
+      <origin xyz="0 0 0" rpy="0 0 0"/>
+      <mass value="0.4"/>
+      <inertia ixx="0.001" ixy="0" ixz="0" iyy="0.001" iyz="0" izz="0.0008"/>
+    </inertial>
+  </link>
   <joint name="neck_pitch" type="revolute">
     <parent link="neck_yaw_link"/><child link="neck_pitch_link"/>
@@ -60,4 +105,10 @@
   </joint>
   <link name="head_link">
+    <!-- ESTIMATED inertia (not measured hardware) -->
+    <inertial>
+      <origin xyz="0 0 0" rpy="0 0 0"/>
+      <mass value="1.2"/>
+      <inertia ixx="0.008" ixy="0" ixz="0" iyy="0.008" iyz="0" izz="0.006"/>
+    </inertial>
     <visual><geometry><mesh filename="${mesh_prefix}/head_shell_front.stl" scale="0.001 0.001 0.001"/></geometry></visual>
     <collision><geometry><cylinder radius="0.04" length="0.08"/></geometry></collision>
@@ -70,4 +121,10 @@
   </joint>
   <link name="left_shoulder_pitch_link">
+    <!-- ESTIMATED inertia (not measured hardware) -->
+    <inertial>
+      <origin xyz="0 0 0" rpy="0 0 0"/>
+      <mass value="1.8"/>
+      <inertia ixx="0.012" ixy="0" ixz="0" iyy="0.012" iyz="0" izz="0.004"/>
+    </inertial>
     <visual><geometry><mesh filename="${mesh_prefix}/upper_arm_shell.stl" scale="0.001 0.001 0.001"/></geometry></visual>
     <collision><geometry><cylinder radius="0.04" length="0.08"/></geometry></collision>
@@ -79,5 +136,12 @@
     <limit lower="-1.4" upper="1.4" effort="1.5" velocity="0.25"/>
   </joint>
-  <link name="left_shoulder_roll_link"/>
+  <link name="left_shoulder_roll_link">
+    <!-- ESTIMATED inertia (not measured hardware) -->
+    <inertial>
+      <origin xyz="0 0 0" rpy="0 0 0"/>
+      <mass value="1.8"/>
+      <inertia ixx="0.012" ixy="0" ixz="0" iyy="0.012" iyz="0" izz="0.004"/>
+    </inertial>
+  </link>
   <joint name="left_shoulder_roll" type="revolute">
     <parent link="left_shoulder_pitch_link"/><child link="left_shoulder_roll_link"/>
@@ -86,5 +150,12 @@
     <limit lower="-0.3" upper="1.5" effort="1.2" velocity="0.25"/>
   </joint>
-  <link name="left_upper_arm_link"/>
+  <link name="left_upper_arm_link">
+    <!-- ESTIMATED inertia (not measured hardware) -->
+    <inertial>
+      <origin xyz="0 0 0" rpy="0 0 0"/>
+      <mass value="1.8"/>
+      <inertia ixx="0.012" ixy="0" ixz="0" iyy="0.012" iyz="0" izz="0.004"/>
+    </inertial>
+  </link>
   <joint name="left_shoulder_yaw" type="revolute">
     <parent link="left_shoulder_roll_link"/><child link="left_upper_arm_link"/>
@@ -94,4 +165,10 @@
   </joint>
   <link name="left_forearm_link">
+    <!-- ESTIMATED inertia (not measured hardware) -->
+    <inertial>
+      <origin xyz="0 0 0" rpy="0 0 0"/>
+      <mass value="1.0"/>
+      <inertia ixx="0.006" ixy="0" ixz="0" iyy="0.006" iyz="0" izz="0.002"/>
+    </inertial>
     <visual><geometry><mesh filename="${mesh_prefix}/forearm_shell.stl" scale="0.001 0.001 0.001"/></geometry></visual>
     <collision><geometry><cylinder radius="0.04" length="0.08"/></geometry></collision>
@@ -103,5 +180,12 @@
     <limit lower="0.0" upper="2.2" effort="1.0" velocity="0.3"/>
   </joint>
-  <link name="left_wrist_yaw_link"/>
+  <link name="left_wrist_yaw_link">
+    <!-- ESTIMATED inertia (not measured hardware) -->
+    <inertial>
+      <origin xyz="0 0 0" rpy="0 0 0"/>
+      <mass value="0.25"/>
+      <inertia ixx="0.0004" ixy="0" ixz="0" iyy="0.0004" iyz="0" izz="0.0002"/>
+    </inertial>
+  </link>
   <joint name="left_wrist_yaw" type="revolute">
     <parent link="left_forearm_link"/><child link="left_wrist_yaw_link"/>
@@ -110,5 +194,12 @@
     <limit lower="-1.4" upper="1.4" effort="0.4" velocity="0.4"/>
   </joint>
-  <link name="left_wrist_pitch_link"/>
+  <link name="left_wrist_pitch_link">
+    <!-- ESTIMATED inertia (not measured hardware) -->
+    <inertial>
+      <origin xyz="0 0 0" rpy="0 0 0"/>
+      <mass value="0.25"/>
+      <inertia ixx="0.0004" ixy="0" ixz="0" iyy="0.0004" iyz="0" izz="0.0002"/>
+    </inertial>
+  </link>
   <joint name="left_wrist_pitch" type="revolute">
     <parent link="left_wrist_yaw_link"/><child link="left_wrist_pitch_link"/>
@@ -118,4 +209,10 @@
   </joint>
   <link name="left_hand_link">
+    <!-- ESTIMATED inertia (not measured hardware) -->
+    <inertial>
+      <origin xyz="0 0 0" rpy="0 0 0"/>
+      <mass value="0.35"/>
+      <inertia ixx="0.0008" ixy="0" ixz="0" iyy="0.0008" iyz="0" izz="0.0004"/>
+    </inertial>
     <visual><geometry><mesh filename="${mesh_prefix}/hand_palm.stl" scale="0.001 0.001 0.001"/></geometry></visual>
     <collision><geometry><cylinder radius="0.04" length="0.08"/></geometry></collision>
@@ -128,4 +225,10 @@
   </joint>
   <link name="left_thumb_link">
+    <!-- ESTIMATED inertia (not measured hardware) -->
+    <inertial>
+      <origin xyz="0 0 0" rpy="0 0 0"/>
+      <mass value="0.05"/>
+      <inertia ixx="5e-05" ixy="0" ixz="0" iyy="5e-05" iyz="0" izz="2e-05"/>
+    </inertial>
     <visual><geometry><mesh filename="${mesh_prefix}/finger_phalanx_proximal.stl" scale="0.001 0.001 0.001"/></geometry></visual>
     <collision><geometry><cylinder radius="0.04" length="0.08"/></geometry></collision>
@@ -138,4 +241,10 @@
   </joint>
   <link name="left_index_link">
+    <!-- ESTIMATED inertia (not measured hardware) -->
+    <inertial>
+      <origin xyz="0 0 0" rpy="0 0 0"/>
+      <mass value="0.05"/>
+      <inertia ixx="5e-05" ixy="0" ixz="0" iyy="5e-05" iyz="0" izz="2e-05"/>
+    </inertial>
     <visual><geometry><mesh filename="${mesh_prefix}/finger_phalanx_proximal.stl" scale="0.001 0.001 0.001"/></geometry></visual>
     <collision><geometry><cylinder radius="0.04" length="0.08"/></geometry></collision>
@@ -148,4 +257,10 @@
   </joint>
   <link name="left_middle_link">
+    <!-- ESTIMATED inertia (not measured hardware) -->
+    <inertial>
+      <origin xyz="0 0 0" rpy="0 0 0"/>
+      <mass value="0.05"/>
+      <inertia ixx="5e-05" ixy="0" ixz="0" iyy="5e-05" iyz="0" izz="2e-05"/>
+    </inertial>
     <visual><geometry><mesh filename="${mesh_prefix}/finger_phalanx_distal.stl" scale="0.001 0.001 0.001"/></geometry></visual>
     <collision><geometry><cylinder radius="0.04" length="0.08"/></geometry></collision>
@@ -158,4 +273,10 @@
   </joint>
   <link name="left_ring_link">
+    <!-- ESTIMATED inertia (not measured hardware) -->
+    <inertial>
+      <origin xyz="0 0 0" rpy="0 0 0"/>
+      <mass value="0.05"/>
+      <inertia ixx="5e-05" ixy="0" ixz="0" iyy="5e-05" iyz="0" izz="2e-05"/>
+    </inertial>
     <visual><geometry><mesh filename="${mesh_prefix}/finger_phalanx_distal.stl" scale="0.001 0.001 0.001"/></geometry></visual>
     <collision><geometry><cylinder radius="0.04" length="0.08"/></geometry></collision>
@@ -168,4 +289,10 @@
   </joint>
   <link name="left_pinky_link">
+    <!-- ESTIMATED inertia (not measured hardware) -->
+    <inertial>
+      <origin xyz="0 0 0" rpy="0 0 0"/>
+      <mass value="0.05"/>
+      <inertia ixx="5e-05" ixy="0" ixz="0" iyy="5e-05" iyz="0" izz="2e-05"/>
+    </inertial>
     <visual><geometry><mesh filename="${mesh_prefix}/finger_phalanx_distal.stl" scale="0.001 0.001 0.001"/></geometry></visual>
     <collision><geometry><cylinder radius="0.04" length="0.08"/></geometry></collision>
@@ -178,4 +305,10 @@
   </joint>
   <link name="right_shoulder_pitch_link">
+    <!-- ESTIMATED inertia (not measured hardware) -->
+    <inertial>
+      <origin xyz="0 0 0" rpy="0 0 0"/>
+      <mass value="1.8"/>
+      <inertia ixx="0.012" ixy="0" ixz="0" iyy="0.012" iyz="0" izz="0.004"/>
+    </inertial>
     <visual><geometry><mesh filename="${mesh_prefix}/upper_arm_shell.stl" scale="0.001 0.001 0.001"/></geometry></visual>
     <collision><geometry><cylinder radius="0.04" length="0.08"/></geometry></collision>
@@ -187,5 +320,12 @@
     <limit lower="-1.4" upper="1.4" effort="1.5" velocity="0.25"/>
   </joint>
-  <link name="right_shoulder_roll_link"/>
+  <link name="right_shoulder_roll_link">
+    <!-- ESTIMATED inertia (not measured hardware) -->
+    <inertial>
+      <origin xyz="0 0 0" rpy="0 0 0"/>
+      <mass value="1.8"/>
+      <inertia ixx="0.012" ixy="0" ixz="0" iyy="0.012" iyz="0" izz="0.004"/>
+    </inertial>
+  </link>
   <joint name="right_shoulder_roll" type="revolute">
     <parent link="right_shoulder_pitch_link"/><child link="right_shoulder_roll_link"/>
@@ -194,5 +334,12 @@
     <limit lower="-1.5" upper="0.3" effort="1.2" velocity="0.25"/>
   </joint>
-  <link name="right_upper_arm_link"/>
+  <link name="right_upper_arm_link">
+    <!-- ESTIMATED inertia (not measured hardware) -->
+    <inertial>
+      <origin xyz="0 0 0" rpy="0 0 0"/>
+      <mass value="1.8"/>
+      <inertia ixx="0.012" ixy="0" ixz="0" iyy="0.012" iyz="0" izz="0.004"/>
+    </inertial>
+  </link>
   <joint name="right_shoulder_yaw" type="revolute">
     <parent link="right_shoulder_roll_link"/><child link="right_upper_arm_link"/>
@@ -202,4 +349,10 @@
   </joint>
   <link name="right_forearm_link">
+    <!-- ESTIMATED inertia (not measured hardware) -->
+    <inertial>
+      <origin xyz="0 0 0" rpy="0 0 0"/>
+      <mass value="1.0"/>
+      <inertia ixx="0.006" ixy="0" ixz="0" iyy="0.006" iyz="0" izz="0.002"/>
+    </inertial>
     <visual><geometry><mesh filename="${mesh_prefix}/forearm_shell.stl" scale="0.001 0.001 0.001"/></geometry></visual>
     <collision><geometry><cylinder radius="0.04" length="0.08"/></geometry></collision>
@@ -211,5 +364,12 @@
     <limit lower="0.0" upper="2.2" effort="1.0" velocity="0.3"/>
   </joint>
-  <link name="right_wrist_yaw_link"/>
+  <link name="right_wrist_yaw_link">
+    <!-- ESTIMATED inertia (not measured hardware) -->
+    <inertial>
+      <origin xyz="0 0 0" rpy="0 0 0"/>
+      <mass value="0.25"/>
+      <inertia ixx="0.0004" ixy="0" ixz="0" iyy="0.0004" iyz="0" izz="0.0002"/>
+    </inertial>
+  </link>
   <joint name="right_wrist_yaw" type="revolute">
     <parent link="right_forearm_link"/><child link="right_wrist_yaw_link"/>
@@ -218,5 +378,12 @@
     <limit lower="-1.4" upper="1.4" effort="0.4" velocity="0.4"/>
   </joint>
-  <link name="right_wrist_pitch_link"/>
+  <link name="right_wrist_pitch_link">
+    <!-- ESTIMATED inertia (not measured hardware) -->
+    <inertial>
+      <origin xyz="0 0 0" rpy="0 0 0"/>
+      <mass value="0.25"/>
+      <inertia ixx="0.0004" ixy="0" ixz="0" iyy="0.0004" iyz="0" izz="0.0002"/>
+    </inertial>
+  </link>
   <joint name="right_wrist_pitch" type="revolute">
     <parent link="right_wrist_yaw_link"/><child link="right_wrist_pitch_link"/>
@@ -226,4 +393,10 @@
   </joint>
   <link name="right_hand_link">
+    <!-- ESTIMATED inertia (not measured hardware) -->
+    <inertial>
+      <origin xyz="0 0 0" rpy="0 0 0"/>
+      <mass value="0.35"/>
+      <inertia ixx="0.0008" ixy="0" ixz="0" iyy="0.0008" iyz="0" izz="0.0004"/>
+    </inertial>
     <visual><geometry><mesh filename="${mesh_prefix}/hand_palm.stl" scale="0.001 0.001 0.001"/></geometry></visual>
     <collision><geometry><cylinder radius="0.04" length="0.08"/></geometry></collision>
@@ -236,4 +409,10 @@
   </joint>
   <link name="right_thumb_link">
+    <!-- ESTIMATED inertia (not measured hardware) -->
+    <inertial>
+      <origin xyz="0 0 0" rpy="0 0 0"/>
+      <mass value="0.05"/>
+      <inertia ixx="5e-05" ixy="0" ixz="0" iyy="5e-05" iyz="0" izz="2e-05"/>
+    </inertial>
     <visual><geometry><mesh filename="${mesh_prefix}/finger_phalanx_proximal.stl" scale="0.001 0.001 0.001"/></geometry></visual>
     <collision><geometry><cylinder radius="0.04" length="0.08"/></geometry></collision>
@@ -246,4 +425,10 @@
   </joint>
   <link name="right_index_link">
+    <!-- ESTIMATED inertia (not measured hardware) -->
+    <inertial>
+      <origin xyz="0 0 0" rpy="0 0 0"/>
+      <mass value="0.05"/>
+      <inertia ixx="5e-05" ixy="0" ixz="0" iyy="5e-05" iyz="0" izz="2e-05"/>
+    </inertial>
     <visual><geometry><mesh filename="${mesh_prefix}/finger_phalanx_proximal.stl" scale="0.001 0.001 0.001"/></geometry></visual>
     <collision><geometry><cylinder radius="0.04" length="0.08"/></geometry></collision>
@@ -256,4 +441,10 @@
   </joint>
   <link name="right_middle_link">
+    <!-- ESTIMATED inertia (not measured hardware) -->
+    <inertial>
+      <origin xyz="0 0 0" rpy="0 0 0"/>
+      <mass value="0.05"/>
+      <inertia ixx="5e-05" ixy="0" ixz="0" iyy="5e-05" iyz="0" izz="2e-05"/>
+    </inertial>
     <visual><geometry><mesh filename="${mesh_prefix}/finger_phalanx_distal.stl" scale="0.001 0.001 0.001"/></geometry></visual>
     <collision><geometry><cylinder radius="0.04" length="0.08"/></geometry></collision>
@@ -266,4 +457,10 @@
   </joint>
   <link name="right_ring_link">
+    <!-- ESTIMATED inertia (not measured hardware) -->
+    <inertial>
+      <origin xyz="0 0 0" rpy="0 0 0"/>
+      <mass value="0.05"/>
+      <inertia ixx="5e-05" ixy="0" ixz="0" iyy="5e-05" iyz="0" izz="2e-05"/>
+    </inertial>
     <visual><geometry><mesh filename="${mesh_prefix}/finger_phalanx_distal.stl" scale="0.001 0.001 0.001"/></geometry></visual>
     <collision><geometry><cylinder radius="0.04" length="0.08"/></geometry></collision>
@@ -276,4 +473,10 @@
   </joint>
   <link name="right_pinky_link">
+    <!-- ESTIMATED inertia (not measured hardware) -->
+    <inertial>
+      <origin xyz="0 0 0" rpy="0 0 0"/>
+      <mass value="0.05"/>
+      <inertia ixx="5e-05" ixy="0" ixz="0" iyy="5e-05" iyz="0" izz="2e-05"/>
+    </inertial>
     <visual><geometry><mesh filename="${mesh_prefix}/finger_phalanx_distal.stl" scale="0.001 0.001 0.001"/></geometry></visual>
     <collision><geometry><cylinder radius="0.04" length="0.08"/></geometry></collision>
@@ -285,5 +488,12 @@
     <limit lower="0.0" upper="1.4" effort="0.15" velocity="0.5"/>
   </joint>
-  <link name="left_hip_yaw_link"/>
+  <link name="left_hip_yaw_link">
+    <!-- ESTIMATED inertia (not measured hardware) -->
+    <inertial>
+      <origin xyz="0 0 0" rpy="0 0 0"/>
+      <mass value="1.5"/>
+      <inertia ixx="0.01" ixy="0" ixz="0" iyy="0.01" iyz="0" izz="0.005"/>
+    </inertial>
+  </link>
   <joint name="left_hip_yaw" type="revolute">
     <parent link="pelvis_link"/><child link="left_hip_yaw_link"/>
@@ -292,5 +502,12 @@
     <limit lower="-0.6" upper="0.6" effort="2.0" velocity="0.25"/>
   </joint>
-  <link name="left_hip_roll_link"/>
+  <link name="left_hip_roll_link">
+    <!-- ESTIMATED inertia (not measured hardware) -->
+    <inertial>
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